Commit message: Added project models

File: model/iiwa7/kuka_iiwa.urdf (robot description, URDF)
Before this commit: robot kuka_iiwa, 8 links, 7 joints
Links:
- link base_link: geometry visual mesh filename=../../../model/iiwa7/meshes/base.obj scale=1 1 1
- link link0: geometry visual mesh filename=../../../model/iiwa7/meshes/link0.obj scale=1 1 1
- link link1: geometry visual mesh filename=../../../model/iiwa7/meshes/link1.obj scale=1 1 1
- link link2: geometry visual mesh filename=../../../model/iiwa7/meshes/link2.obj scale=1 1 1
- link link3: geometry visual mesh filename=../../../model/iiwa7/meshes/link3.obj scale=1 1 1
- link link4: geometry visual mesh filename=../../../model/iiwa7/meshes/link4.obj scale=1 1 1
- link link5: geometry visual mesh filename=../../../model/iiwa7/meshes/link5.obj scale=1 1 1
- link link6: geometry visual mesh filename=../../../model/iiwa7/meshes/link6.obj scale=1 1 1
